File: Weather-Station.kicad_pcb (KiCad board)
At the start: 2 copper layers, 160 x 140 mm, 7 parts, among them J1 Conn_01x22, J2 Conn_01x22, J3 CN2, J4 CN3, J5 Conn_02x22_Odd_Even, J6 Conn_01x22, J7 Conn_01x06

Commit message: PCB done
Routing:
- net GND: track 142.1 -> 119.5 mm, vias 168 -> 176
Changed lines of the file:
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@@
 		(capping no)
 		(filling no)
-		(zone_defaults)
 		(aux_axis_origin 157.48 208.28)
 		(grid_origin 157.48 208.28)
@@
 	)
 	(gr_text "Weather Station V1.0"
-		(at 162.56 203.2 0)
+		(at 167.074405 201.475029 0)
 		(layer "F.SilkS")
 		(effects
 			(font
-				(size 10 5)
+				(size 5 3)
 				(bold yes)
 			)
@@
 	)
 	(segment
-		(start 174.54 121.92)
-		(end 174.58 121.88)
-		(width 1)
-		(layer "F.Cu")
-		(net "GND")
-	)
-	(segment
 		(start 266.7 132.10208)
 		(end 278.10792 132.10208)
@@
 	)
 	(segment
-		(start 171.45 137.16)
-		(end 174.7 137.16)
-		(width 1)
-		(layer "F.Cu")
-		(net "GND")
-	)
-	(segment
-		(start 243.47 76.17)
-		(end 243.48 76.18)
-		(width 2)
-		(layer "F.Cu")
-		(net "GND")
-	)
-	(segment
 		(start 312.39792 78.74)
 		(end 312.42 78.76208)
@@
 	)
 	(segment
-		(start 251.09 73.68)
-		(end 251.09 76.37)
-		(width 2)
-		(layer "F.Cu")
-		(net "GND")
-	)
-	(segment
 		(start 229.87 124.46)
 		(end 226.06 124.46)
@@
 	)
 	(segment
-		(start 251.09 76.37)
-		(end 251.08 76.38)
-		(width 2)
-		(layer "F.Cu")
-		(net "GND")
-	)
-	(segment
 		(start 174.7 137.16)
 		(end 174.78 137.08)
@@
 	)
 	(segment
-		(start 243.47 73.68)
-		(end 243.47 76.17)
-		(width 2)
-		(layer "F.Cu")
-		(net "GND")
-	)
-	(segment
 		(start 278.10792 132.10208)
 		(end 278.13 132.08)
@@
 	)
 	(segment
-		(start 168.91 137.16)
-		(end 166.5 137.16)
-		(width 1)
-		(layer "F.Cu")
-		(net "GND")
-	)
-	(segment
-		(start 171.45 121.92)
-		(end 174.54 121.92)
-		(width 1)
-		(layer "F.Cu")
-		(net "GND")
-	)
-	(segment
 		(start 232.41 137.16)
 		(end 232.43 137.18)
@@
 	)
 	(segment
-		(start 171.45 139.7)
-		(end 174.5 139.7)
-		(width 1)
-		(layer "F.Cu")
-		(net "GND")
-	)
-	(segment
 		(start 312.42 132.08)
 		(end 312.42 132.10208)
@@
 	)
 	(via
-		(at 180.34 203.2)
+		(at 182.314405 204.015029)
 		(size 1)
 		(drill 0.5)
@@
 	)
 	(via
+		(at 221.98 105.78)
+		(size 1)
+		(drill 0.5)
+		(layers "F.Cu" "B.Cu")
+		(free yes)
+		(net "GND")
+	)
+	(via
 		(at 221.330668 141.808763)
 		(size 1)
@@
 	)
 	(via
+		(at 218.88 128.28)
+		(size 1)
+		(drill 0.5)
+		(layers "F.Cu" "B.Cu")
+		(free yes)
+		(net "GND")
+	)
+	(via
 		(at 205.74 116.84)
 		(size 1)
@@
 	)
 	(via
+		(at 218.88 110.08)
+		(size 1)
+		(drill 0.5)
+		(layers "F.Cu" "B.Cu")
+		(free yes)
+		(net "GND")
+	)
+	(via
 		(at 190.5 124.46)
 		(size 1)
@@
 	)
 	(via
+		(at 218.88 120.68)
+		(size 1)
+		(drill 0.5)
+		(layers "F.Cu" "B.Cu")
+		(free yes)
+		(net "GND")
+	)
+	(via
 		(at 269.24 160.02)
 		(size 1)
@@
 	)
 	(via
+		(at 254.58 109.58)
+		(size 1)
+		(drill 0.5)
+		(layers "F.Cu" "B.Cu")
+		(free yes)
+		(net "GND")
+	)
+	(via
+		(at 249.28 105.78)
+		(size 1)
+		(drill 0.5)
+		(layers "F.Cu" "B.Cu")
+		(free yes)
+		(net "GND")
+	)
+	(via
 		(at 314.96 172.72)
 		(size 1)
@@
 	)
 	(via
+		(at 243.28 108.18)
+		(size 1)
+		(drill 0.5)
+		(layers "F.Cu" "B.Cu")
+		(free yes)
+		(net "GND")
+	)
+	(via
 		(at 174.68 139.88)
 		(size 1)
@@
 	)
 	(via
+		(at 231.88 105.38)
+		(size 1)
+		(drill 0.5)
+		(layers "F.Cu" "B.Cu")
+		(free yes)
+		(net "GND")
+	)
+	(via
 		(at 185.42 81.28)
 		(size 1)
@@
 	)
 	(segment
-		(start 243.47 76.37)
-		(end 243.48 76.38)
-		(width 2)
-		(layer "B.Cu")
-		(net "GND")
-	)
-	(segment
 		(start 174.88 137.18)
 		(end 174.86 137.16)
@@
 	)
 	(segment
-		(start 251.09 76.39)
-		(end 251.18 76.48)
-		(width 2)
-		(layer "B.Cu")
-		(net "GND")
-	)
-	(segment
 		(start 232.41 137.16)
 		(end 234.1 137.16)
@@
 	)
 	(segment
-		(start 251.09 73.68)
-		(end 251.09 76.39)
-		(width 2)
-		(layer "B.Cu")
-		(net "GND")
-	)
-	(segment
 		(start 171.45 121.92)
 		(end 174.94 121.92)
@@
 	)
 	(segment
-		(start 243.47 73.68)
-		(end 243.47 76.37)
-		(width 2)
-		(layer "B.Cu")
-		(net "GND")
-	)
-	(segment
 		(start 171.45 137.16)
 		(end 171.45 139.7)
@@
 	)
 	(segment
-		(start 222.38 132.21)
-		(end 229.87 139.7)
+		(start 264.16 116.86208)
+		(end 244.66208 116.86208)
 		(width 0.5)
 		(layer "B.Cu")
@@
 	)
 	(segment
-		(start 264.16 116.86208)
-		(end 244.66208 116.86208)
+		(start 222.38 130.08)
+		(end 227.08 134.78)
+		(width 0.5)
+		(layer "B.Cu")
+		(net "/DISP_CS")
+	)
+	(segment
+		(start 222.38 111.88)
+		(end 222.38 130.08)
+		(width 0.5)
+		(layer "B.Cu")
+		(net "/DISP_CS")
+	)
+	(segment
+		(start 227.08 136.91)
+		(end 229.87 139.7)
 		(width 0.5)
 		(layer "B.Cu")
@@
 	)
 	(segment
-		(start 222.38 111.88)
-		(end 222.38 132.21)
+		(start 244.66208 116.86208)
+		(end 236.28 108.48)
 		(width 0.5)
 		(layer "B.Cu")
@@
 	)
 	(segment
-		(start 225.78 108.48)
-		(end 222.38 111.88)
+		(start 227.08 134.78)
+		(end 227.08 136.91)
 		(width 0.5)
 		(layer "B.Cu")
@@
 	)
 	(segment
-		(start 229.79 139.78)
-		(end 229.87 139.7)
+		(start 225.78 108.48)
+		(end 222.38 111.88)
 		(width 0.5)
 		(layer "B.Cu")
@@
 	)
 	(segment
-		(start 244.66208 116.86208)
-		(end 236.28 108.48)
+		(start 229.79 139.78)
+		(end 229.87 139.7)
 		(width 0.5)
 		(layer "B.Cu")
@@
 	)
 	(segment
-		(start 237.58 107.18)
-		(end 224.08 107.18)
+		(start 220.68 110.58)
+		(end 220.68 132.08)
 		(width 0.5)
 		(layer "B.Cu")
@@
 	)
 	(segment
-		(start 229.18 144.78)
-		(end 229.87 144.78)
+		(start 264.16 111.78208)
+		(end 264.06208 111.88)
 		(width 0.5)
 		(layer "B.Cu")
@@
 	)
 	(segment
-		(start 220.68 110.58)
-		(end 220.68 132.08)
+		(start 264.06208 111.88)
+		(end 242.28 111.88)
 		(width 0.5)
 		(layer "B.Cu")
@@
 	)
 	(segment
-		(start 224.08 107.18)
-		(end 220.68 110.58)
+		(start 224.28 135.68)
+		(end 224.28 139.19)
 		(width 0.5)
 		(layer "B.Cu")
@@
 	)
 	(segment
-		(start 220.68 132.08)
-		(end 222.88 134.28)
+		(start 237.58 107.18)
+		(end 224.08 107.18)
 		(width 0.5)
 		(layer "B.Cu")
@@
 	)
 	(segment
-		(start 264.06208 111.88)
-		(end 242.28 111.88)
+		(start 229.18 144.78)
+		(end 229.87 144.78)
 		(width 0.5)
 		(layer "B.Cu")
@@
 	)
 	(segment
-		(start 242.28 111.88)
-		(end 237.58 107.18)
+		(start 220.68 132.08)
+		(end 224.28 135.68)
 		(width 0.5)
 		(layer "B.Cu")
@@
 	)
 	(segment
-		(start 222.88 134.28)
-		(end 222.88 137.79)
+		(start 242.28 111.88)
+		(end 237.58 107.18)
 		(width 0.5)
 		(layer "B.Cu")
@@
 	)
 	(segment
-		(start 264.16 111.78208)
-		(end 264.06208 111.88)
+		(start 224.28 139.19)
+		(end 229.87 144.78)
 		(width 0.5)
 		(layer "B.Cu")
@@
 	)
 	(segment
-		(start 222.88 137.79)
-		(end 229.87 144.78)
+		(start 224.08 107.18)
+		(end 220.68 110.58)
 		(width 0.5)
 		(layer "B.Cu")
@@
 		(polygon
 			(pts
-				(xy 279.38 80.88) (xy 299.78 80.88) (xy 299.78 77.58) (xy 317.48 77.58) (xy 317.48 68.28) (xy 270.58 68.28)
-				(xy 270.58 77.48) (xy 279.38 77.48)
+				(xy 278.94 80.88) (xy 297.78 80.88) (xy 297.78 77.58) (xy 316.98 77.58) (xy 316.98 68.28) (xy 270.58 68.28)
+				(xy 270.58 77.48) (xy 278.94 77.48)
 			)
 		)
